File: CM4_2.kicad_pcb (KiCad board)
At the start: 4 copper layers, 90 x 75 mm, 28 parts, among them J1 Bus_PCI_Express_Mini, J10 PCIE_USB_D-/D+, J11 V_IN1, J12 V_IN2, J17 GPIO_V, J2 USB_A, J20 Controll Connector, J3 USB_HUB, J30 GPIO Connector, J4 USB_B_Micro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

Commit message: Some tracks rerouted, MicroUSB moved
Parts:
- moved J4 61.7 mm to (498.6, 296.2)
- moved J42 0.30 mm to (547.1, 311.8)
- moved J10 0.26 mm to (553.5, 311.8)
Routing:
- net /USB2_N: track 65.3 -> 104.2 mm
- net /USB2_P: track 66.1 -> 104.8 mm
- net +5V_USB_IN: track 196.6 -> 162.1 mm
- net GND: track 7.17 -> 15.9 mm, vias 2 -> 7
- net 3V3_PCIE: track 67.4 -> 60.1 mm
- net +5V_USB: track 89.5 -> 95.8 mm
- net /Eth_P1_P: track 61.0 -> 56.6 mm
- net /Eth_P1_N: track 61.0 -> 56.8 mm
- net /HDMI0_SCL: track 76.9 -> 80.2 mm
- net /HDMI0_HOTPLUG: track 78.7 -> 81.6 mm
- net /HDMI0_SDA: track 80.3 -> 82.0 mm
- net +5V_HDMI: track 84.0 -> 82.7 mm
- net /SD_DAT2: track 42.4 -> 43.5 mm
- net /HDMI0_CEC: track 73.0 -> 74.0 mm
- net /SD_CMD: track 80.2 -> 81.1 mm
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Other:
- board text added: "Description on backside"
- board text added: "J20"
