File: CM4_2.kicad_pcb (KiCad board)
At the start: 4 copper layers, 90 x 75 mm, 28 parts, among them J1 Bus_PCI_Express_Mini, J10 PCIE_USB_D-/D+, J11 V_IN1, J12 V_IN2, J17 GPIO_V, J2 USB_A, J20 Controll Connector, J3 USB_HUB, J30 GPIO Connector, J4 USB_B_Micro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

Commit message: R2 to R1, C2 to C1
Parts:
- renumbered C2 to C1, R2 to R1
Changed lines of the file:
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@@
     (property "Sheet name" "")
     (attr smd)
-    (fp_text reference "R2" (at 3.556 -0.127) (layer "F.SilkS")
+    (fp_text reference "R1" (at 3.556 -0.127) (layer "F.SilkS")
       (effects (font (size 1 1) (thickness 0.15)))
     )
@@
     (property "Sheet name" "")
     (attr smd)
-    (fp_text reference "C2" (at -3.429 0) (layer "F.SilkS")
-      (effects (font (size 1 1) (thickness 0.15)))
-    )
+    (fp_text reference "C1" (at -3.429 0) (layer "F.SilkS")
+      (effects (font (size 1 1) (thickness 0.15)))
+    )

Commit message: Minor
Parts:
- moved J40 0.89 mm to (495.0, 331.9)
Routing:
- net /Eth_P1_N: track 56.8 -> 32.8 mm
- net /Eth_P1_P: track 56.6 -> 34.8 mm
- net /SD_DAT3: track 40.6 -> 52.0 mm
- net /SD_DAT2: track 43.5 -> 53.9 mm
- net GND: track 15.9 -> 9.76 mm, vias 7 -> 21
- net /PCIe_nRST: track 28.6 -> 25.5 mm
- net /SD_DAT0: track 57.0 -> 55.0 mm
- net /SD_DAT1: track 47.5 -> 46.2 mm
- net 1.8V_CM4: track 24.2 -> 25.5 mm
- net GPIO14: track 14.5 -> 13.8 mm

Commit message: v1.01
Parts:
- removed ? (x6): , 
- removed J41: GND, Connector_PinHeader_2.54mm:PinHeader_1x01_P2.54mm_Vertical
- J17: footprint Connector_PinHeader_2.54mm:PinHeader_1x03_P2.54mm_Vertical -> Connector_PinHeader_2.54mm:PinHeader_1x03_P2.54mm_Vertical_SMD_Pin1Right; moved to B.Cu
- J30: value GPIO Connector -> Conn_01x07_Female; footprint Connector_PinHeader_2.54mm:PinHeader_1x06_P2.54mm_Vertical -> Connector_PinSocket_2.54mm:PinSocket_1x07_P2.54mm_Vertical
- moved J17 3.29 mm to (495.0, 352.9), turned to 180 degrees
- moved J40 0.13 mm to (495.0, 331.7)
- moved J30 0.06 mm to (487.6, 320.6)
Connections:
- J17 pad 1: 1.8V_CM4 -> 3.3V_CM4
- J17 pad 2: 3.3V_CM4 -> GPIO_VREF
- J17 pad 3: GPIO_VREF -> 1.8V_CM4
Routing:
- net 3.3V_CM4: track 74.0 -> 61.9 mm, vias 2 -> 3
- net 1.8V_CM4: track 25.5 -> 31.5 mm, vias 0 -> 1
- net +5V_USB: track 95.8 -> 90.3 mm
- net /Eth_P1_N: track 32.8 -> 34.8 mm
- net GND: track 9.76 -> 7.83 mm, vias 21 -> 84
- net /SD_PWR_ON: track 54.1 -> 52.6 mm
- net +5V_HDMI: track 82.7 -> 81.4 mm
- net /HDMI0_HOTPLUG: track 81.6 -> 80.4 mm
- net GPIO_VREF: track 28.4 -> 27.2 mm, vias 0 -> 1
- net PI_N_LED: track 4.05 -> 5.07 mm
- net /SD_DAT3: track 52.0 -> 52.9 mm
- net PI_POWER_LED: track 14.6 -> 15.4 mm
- net /USB2_N: track 103.8 -> 104.5 mm
- net /USB2_P: track 104.8 -> 105.5 mm
- net /SD_CLK: track 58.2 -> 58.9 mm
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Other:
- outline, holes or cut-outs redrawn
- board text added: "+1.8"
- board text added: "+3.3"
- board text added: "GPIO_Vref"
- board text added: "HDMI"
- board text added: "Pinout on backside"
- board text added: "Raspberry PI CM4 NAS MiniPCIE V 1.01 (Not Tested) https://github.com/olvint/CM4-NAS-MiniPCIE"
- board text removed: "+1.8V +3.3V GPIO_V"
- board text removed: "Description on backside"
- board text removed: "Raspberry PI CM4 NAS MiniPCIE V 1.0 (Not Tested) https://github.com/olvint/CM4-NAS-MiniPCIE"
