File: CM4_2_Backup.kicad_pcb (KiCad board)
At the start: 4 copper layers, 90 x 75 mm, 25 parts, among them J1 Bus_PCI_Express_Mini, J10 PCIE_USB_D-/D+, J11 V_IN1, J12 V_IN2, J17 GPIO_V, J2 USB_A, J20 Controll Connector, J3 USB_HUB, J30 Conn_01x07_Female, J4 USB_B_Micro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

Commit message: Drill Holes
Parts:
- removed REF** (x2): MountingHole_3.2mm_M3, MountingHole:MountingHole_3.2mm_M3
- removed REF** (x2): MountingHole_3.2mm_M3_ISO7380_Pad, MountingHole:MountingHole_3.2mm_M3_ISO7380_Pad
Routing:
- net +5V_USB: track 91.7 -> 90.3 mm
Other:
- outline, holes or cut-outs redrawn
Changed lines of the file:
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@@
     )
-  )
-  (footprint "MountingHole:MountingHole_3.2mm_M3" (layer "F.Cu")
-    (at 490 360)
-    (descr "Mounting Hole 3.2mm, no annular, M3")
-    (tags "mounting hole 3.2mm no annular m3")
-    (attr exclude_from_pos_files exclude_from_bom)
-    (fp_text reference "REF**" (at 4.7 3.4) (layer "F.Fab")
-      (effects (font (size 1 1) (thickness 0.15)))
-    )
-    (fp_text value "MountingHole_3.2mm_M3" (at 0 4.2) (layer "F.Fab")
-      (effects (font (size 1 1) (thickness 0.15)))
-    )
-    (fp_circle (center 0 0) (end 3.2 0) (layer "Cmts.User") (width 0.15) (fill none))
-    (fp_circle (center 0 0) (end 3.45 0) (layer "F.CrtYd") (width 0.05) (fill none))
-    (pad "1" np_thru_hole circle (at 0 0) (size 3.2 3.2) (drill 3.2) (layers *.Cu *.Mask))
   )
   (footprint "Resistor_SMD:R_0805_2012Metric" (layer "F.Cu")
@@
     )
   )
-  (footprint "MountingHole:MountingHole_3.2mm_M3" (layer "F.Cu")
-    (at 570 360)
-    (descr "Mounting Hole 3.2mm, no annular, M3")
-    (tags "mounting hole 3.2mm no annular m3")
-    (attr exclude_from_pos_files exclude_from_bom)
-    (fp_text reference "REF**" (at 0 -4.2) (layer "F.Fab")
-      (effects (font (size 1 1) (thickness 0.15)))
-    )
-    (fp_text value "MountingHole_3.2mm_M3" (at 0 4.2) (layer "F.Fab")
-      (effects (font (size 1 1) (thickness 0.15)))
-    )
-    (fp_text user "${REFERENCE}" (at 0.3 0) (layer "F.Fab")
-      (effects (font (size 1 1) (thickness 0.15)))
-    )
-    (fp_circle (center 0 0) (end 3.2 0) (layer "Cmts.User") (width 0.15) (fill none))
-    (fp_circle (center 0 0) (end 3.45 0) (layer "F.CrtYd") (width 0.05) (fill none))
-    (pad "1" np_thru_hole circle (at 0 0) (size 3.2 3.2) (drill 3.2) (layers *.Cu *.Mask))
-  )
   (footprint "Resistor_SMD:R_0805_2012Metric" (layer "F.Cu")
     (at 560.2875 356.11)
@@
       (rotate (xyz 0 0 0))
     )
-  )
-  (footprint "MountingHole:MountingHole_3.2mm_M3_ISO7380_Pad" (layer "F.Cu")
-    (at 568.590489 342.747554)
-    (descr "Mounting Hole 3.2mm, M3, ISO7380")
-    (tags "mounting hole 3.2mm m3 iso7380")
-    (attr exclude_from_pos_files exclude_from_bom)
-    (fp_text reference "REF**" (at 9.147209 0.270729) (layer "F.SilkS")
-      (effects (font (size 1 1) (thickness 0.15)))
-    )
-    (fp_text value "MountingHole_3.2mm_M3_ISO7380_Pad" (at 21.593704 2.473985) (layer "F.Fab")
-      (effects (font (size 1 1) (thickness 0.15)))
-    )
-    (fp_text user "${REFERENCE}" (at 0.3 0) (layer "F.Fab")
-      (effects (font (size 1 1) (thickness 0.15)))
-    )
-    (fp_circle (center 0 0) (end 2.85 0) (layer "Cmts.User") (width 0.15) (fill none))
-    (fp_circle (center 0 0) (end 3.1 0) (layer "F.CrtYd") (width 0.05) (fill none))
-    (pad "1" thru_hole circle (at 0 0) (size 5.7 5.7) (drill 3.2) (layers *.Cu *.Mask))
-  )
-  (footprint "MountingHole:MountingHole_3.2mm_M3_ISO7380_Pad" (layer "F.Cu")
-    (at 568.593883 318.583037)
-    (descr "Mounting Hole 3.2mm, M3, ISO7380")
-    (tags "mounting hole 3.2mm m3 iso7380")
-    (attr exclude_from_pos_files exclude_from_bom)
-    (fp_text reference "REF**" (at 9.147209 0.270729) (layer "F.SilkS")
-      (effects (font (size 1 1) (thickness 0.15)))
-    )
-    (fp_text value "MountingHole_3.2mm_M3_ISO7380_Pad" (at 21.593704 2.473985) (layer "F.Fab")
-      (effects (font (size 1 1) (thickness 0.15)))
-    )
-    (fp_text user "${REFERENCE}" (at 0.3 0) (layer "F.Fab")
-      (effects (font (size 1 1) (thickness 0.15)))
-    )
-    (fp_circle (center 0 0) (end 2.85 0) (layer "Cmts.User") (width 0.15) (fill none))
-    (fp_circle (center 0 0) (end 3.1 0) (layer "F.CrtYd") (width 0.05) (fill none))
-    (pad "1" thru_hole circle (at 0 0) (size 5.7 5.7) (drill 3.2) (layers *.Cu *.Mask))
   )
   (footprint "Connector_PinHeader_2.54mm:PinHeader_1x01_P2.54mm_Vertical" (layer "F.Cu")
@@
   (gr_line (start 490 365) (end 565 365) (layer "Edge.Cuts") (width 0.1))
   (gr_arc (start 490 295) (end 485 295) (angle 90) (layer "Edge.Cuts") (width 0.1))
+  (gr_circle (center 568.604886 318.623459) (end 570.204886 318.623459) (layer "Edge.Cuts") (width 0.1) (fill solid))
+  (gr_circle (center 570 360) (end 571.6 360) (layer "Edge.Cuts") (width 0.1) (fill solid))
   (gr_line (start 485 360) (end 485 295) (layer "Edge.Cuts") (width 0.1))
+  (gr_circle (center 568.567325 342.833718) (end 570.167325 342.833718) (layer "Edge.Cuts") (width 0.1) (fill solid))
+  (gr_circle (center 532 307) (end 533.6 307) (layer "Edge.Cuts") (width 0.1) (fill solid))
   (gr_line (start 575 360) (end 575 295) (layer "Edge.Cuts") (width 0.1))
   (gr_arc (start 570 295) (end 575 295) (angle -90) (layer "Edge.Cuts") (width 0.1))
   (gr_line (start 570 290) (end 490 290) (layer "Edge.Cuts") (width 0.1))
   (gr_arc (start 490 360) (end 485 360) (angle -90) (layer "Edge.Cuts") (width 0.1))
+  (gr_circle (center 490 360) (end 491.6 360) (layer "Edge.Cuts") (width 0.1) (fill solid))
   (gr_text "+3.3" (at 498.475 349.631) (layer "B.SilkS")
     (effects (font (size 1 1) (thickness 0.15)) (justify mirror))
@@
   (via (at 563 351.5) (size 0.8) (drill 0.45) (layers "F.Cu" "B.Cu") (free) (net 12))
   (via (at 565 351.5) (size 0.8) (drill 0.45) (layers "F.Cu" "B.Cu") (free) (net 12))
+  (segment (start 551.3152 306) (end 545.38 306) (width 1) (layer "B.Cu") (net 12))
+  (segment (start 572.229297 309.989297) (end 568.232588 305.992588) (width 1) (layer "B.Cu") (net 12))
+  (segment (start 549.618992 304.303792) (end 551.3152 306) (width 1) (layer "B.Cu") (net 12))
+  (segment (start 572.229297 344.229297) (end 572.229297 309.989297) (width 1) (layer "B.Cu") (net 12))
+  (segment (start 558.007412 305.992588) (end 558 306) (width 1) (layer "B.Cu") (net 12))
+  (segment (start 549.618992 300.788592) (end 549.618992 304.303792) (width 1) (layer "B.Cu") (net 12))
   (segment (start 558 306) (end 551.3152 306) (width 1) (layer "B.Cu") (net 12))
-  (segment (start 558.007412 305.992588) (end 558 306) (width 1) (layer "B.Cu") (net 12))
-  (segment (start 551.3152 306) (end 545.38 306) (width 1) (layer "B.Cu") (net 12))
-  (segment (start 549.618992 304.303792) (end 551.3152 306) (width 1) (layer "B.Cu") (net 12))
-  (segment (start 566.284956 351.5) (end 572.964622 344.820334) (width 1) (layer "B.Cu") (net 12))
-  (segment (start 565 351.5) (end 566.284956 351.5) (width 1) (layer "B.Cu") (net 12))
-  (segment (start 549.618992 300.788592) (end 549.618992 304.303792) (width 1) (layer "B.Cu") (net 12))
   (segment (start 545.38 306) (end 542.15 302.77) (width 1) (layer "B.Cu") (net 12))
-  (segment (start 572.964622 344.820334) (end 572.964622 310.724622) (width 1) (layer "B.Cu") (net 12))
-  (segment (start 572.964622 310.724622) (end 568.232588 305.992588) (width 1) (layer "B.Cu") (net 12))
   (segment (start 568.232588 305.992588) (end 558.007412 305.992588) (width 1) (layer "B.Cu") (net 12))
+  (segment (start 572.229297 344.270703) (end 572.229297 344.229297) (width 1) (layer "B.Cu") (net 12))
+  (segment (start 565 351.5) (end 572.229297 344.270703) (width 1) (layer "B.Cu") (net 12))
   (segment (start 545.225152 347.785802) (end 545.267171 347.743783) (width 0.175006) (layer "F.Cu") (net 13))
   (segment (start 546.131386 347.837044) (end 546.190437 347.843697) (width 0.175006) (layer "F.Cu") (net 13))
